File: Conception/Communication.kicad_sch (KiCad schematic)
At the start: 0 parts

Commit message: MAJ
Other:
- company: AstroMonkeys -> (none)
Changed lines of the file:
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@@
 (kicad_sch (version 20211123) (generator eeschema)
   (paper "A4")
-  (title_block
-    (rev "0.1")
-    (company "AstroMonkeys")
-  )
 )
