File: Conception/Connecteurs.kicad_sch (KiCad schematic)
At the start: 0 parts

Commit message: MAJ
Parts:
- added J? (x5): Conn_01x02_Male, Connector_PinSocket_2.54mm:PinSocket_1x02_P2.54mm_Horizontal, symbol Connector:Conn_01x02_Male
- added J? (x2): Conn_01x04_Male, Connector_PinHeader_2.54mm:PinHeader_1x04_P2.54mm_Horizontal, symbol Connector:Conn_01x04_Male
- added J? (x2): Conn_01x02_Male, Connector_Phoenix_MC_HighVoltage:PhoenixContact_MC_1,5_2-G-5.08_1x02_P5.08mm_Horizontal, symbol Connector:Conn_01x02_Male
Connections:
- new net GND: J?.2 (Pin_2), J?.2 (Pin_2), J?.4 (Pin_4), J?.4 (Pin_4)
Other:
- note added: "ALIMENTATION"
- note added: "CAN"
- note added: "MOTEUR"
- note added: "ROUE CODEUSE"
Changed lines of the file:
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@@
     (company "AstroMonkeys")
   )
+  (wire (pts (xy 161.29 44.45) (xy 161.29 46.99))
+    (stroke (width 0) (type default) (color 0 0 0 0))
+  )
+  (polyline (pts (xy 198.12 73.66) (xy 135.89 73.66))
+    (stroke (width 0) (type default) (color 0 0 0 0))
+  )
+  (polyline (pts (xy 73.66 73.66) (xy 73.66 144.78))
+    (stroke (width 0) (type default) (color 0 0 0 0))
+  )
+  (polyline (pts (xy 198.12 12.7) (xy 198.12 73.66))
+    (stroke (width 0) (type default) (color 0 0 0 0))
+  )
+  (polyline (pts (xy 73.66 144.78) (xy 11.43 144.78))
+    (stroke (width 0) (type default) (color 0 0 0 0))
+  )
+  (polyline (pts (xy 73.66 12.7) (xy 73.66 73.66))
+    (stroke (width 0) (type default) (color 0 0 0 0))
+  )
+  (polyline (pts (xy 73.66 73.66) (xy 11.43 73.66))
+    (stroke (width 0) (type default) (color 0 0 0 0))
+  )
+  (wire (pts (xy 39.37 60.96) (xy 39.37 63.5))
+    (stroke (width 0) (type default) (color 0 0 0 0))
+  )
+  (wire (pts (xy 39.37 41.91) (xy 39.37 44.45))
+    (stroke (width 0) (type default) (color 0 0 0 0))
+  )
+  (wire (pts (xy 36.83 41.91) (xy 39.37 41.91))
+    (stroke (width 0) (type default) (color 0 0 0 0))
+  )
+  (wire (pts (xy 36.83 60.96) (xy 39.37 60.96))
+    (stroke (width 0) (type default) (color 0 0 0 0))
+  )
+  (polyline (pts (xy 135.89 12.7) (xy 135.89 73.66))
+    (stroke (width 0) (type default) (color 0 0 0 0))
+  )
+  (wire (pts (xy 158.75 44.45) (xy 161.29 44.45))
+    (stroke (width 0) (type default) (color 0 0 0 0))
+  )
+  (polyline (pts (xy 135.89 73.66) (xy 73.66 73.66))
+    (stroke (width 0) (type default) (color 0 0 0 0))
+  )
+  (wire (pts (xy 158.75 63.5) (xy 161.29 63.5))
+    (stroke (width 0) (type default) (color 0 0 0 0))
+  )
+  (wire (pts (xy 161.29 63.5) (xy 161.29 66.04))
+    (stroke (width 0) (type default) (color 0 0 0 0))
+  )
+  (text "CAN\n" (at 30.48 83.82 180)
+    (effects (font (size 4 4)) (justify left bottom))
+  )
+  (text "MOTEUR\n" (at 91.44 22.86 180)
+    (effects (font (size 4 4)) (justify left bottom))
+  )
+  (text "ROUE CODEUSE" (at 144.78 22.86 180)
+    (effects (font (size 4 4)) (justify left bottom))
+  )
+  (text "ALIMENTATION" (at 20.32 22.86 180)
+    (effects (font (size 4 4)) (justify left bottom))
+  )
+  (symbol (lib_id "Connector:Conn_01x02_Male") (at 31.75 118.11 0) (unit 1)
+    (in_bom yes) (on_board yes) (fields_autoplaced)
+    (property "Reference" "J?" (id 0) (at 32.385 113.03 0))
+    (property "Value" "Conn_01x02_Male" (id 1) (at 32.385 115.57 0))
+    (property "Footprint" "Connector_PinSocket_2.54mm:PinSocket_1x02_P2.54mm_Horizontal" (id 2) (at 31.75 118.11 0)
+      (effects (font (size 1.27 1.27)) hide)
+    )
+    (property "Datasheet" "~" (id 3) (at 31.75 118.11 0)
+      (effects (font (size 1.27 1.27)) hide)
+    )
+    (pin "1")
+    (pin "2")
+  )
+  (symbol (lib_id "power:GND") (at 39.37 63.5 0) (unit 1)
+    (in_bom yes) (on_board yes) (fields_autoplaced)
+    (property "Reference" "#PWR?" (id 0) (at 39.37 69.85 0)
+      (effects (font (size 1.27 1.27)) hide)
+    )
+    (property "Value" "GND" (id 1) (at 39.37 68.58 0))
+    (property "Footprint" "" (id 2) (at 39.37 63.5 0)
+      (effects (font (size 1.27 1.27)) hide)
+    )
+    (property "Datasheet" "" (id 3) (at 39.37 63.5 0)
+      (effects (font (size 1.27 1.27)) hide)
+    )
+    (pin "1")
+  )
+  (symbol (lib_id "Connector:Conn_01x02_Male") (at 31.75 137.16 0) (unit 1)
+    (in_bom yes) (on_board yes)
+    (property "Reference" "J?" (id 0) (at 32.385 132.08 0))
+    (property "Value" "Conn_01x02_Male" (id 1) (at 32.385 134.62 0))
+    (property "Footprint" "Connector_PinSocket_2.54mm:PinSocket_1x02_P2.54mm_Horizontal" (id 2) (at 31.75 137.16 0)
+      (effects (font (size 1.27 1.27)) hide)
+    )
+    (property "Datasheet" "~" (id 3) (at 31.75 137.16 0)
+      (effects (font (size 1.27 1.27)) hide)
+    )
+    (pin "1")
+    (pin "2")
+  )
+  (symbol (lib_id "power:GND") (at 39.37 44.45 0) (unit 1)
+    (in_bom yes) (on_board yes) (fields_autoplaced)
+    (property "Reference" "#PWR?" (id 0) (at 39.37 50.8 0)
+      (effects (font (size 1.27 1.27)) hide)
+    )
+    (property "Value" "GND" (id 1) (at 39.37 49.53 0))
+    (property "Footprint" "" (id 2) (at 39.37 44.45 0)
+      (effects (font (size 1.27 1.27)) hide)
+    )
+    (property "Datasheet" "" (id 3) (at 39.37 44.45 0)
+      (effects (font (size 1.27 1.27)) hide)
+    )
+    (pin "1")
+  )
+  (symbol (lib_id "Connector:Conn_01x04_Male") (at 153.67 39.37 0) (unit 1)
+    (in_bom yes) (on_board yes) (fields_autoplaced)
+    (property "Reference" "J?" (id 0) (at 154.305 31.75 0))
+    (property "Value" "Conn_01x04_Male" (id 1) (at 154.305 34.29 0))
+    (property "Footprint" "Connector_PinHeader_2.54mm:PinHeader_1x04_P2.54mm_Horizontal" (id 2) (at 153.67 39.37 0)
+      (effects (font (size 1.27 1.27)) hide)
+    )
+    (property "Datasheet" "~" (id 3) (at 153.67 39.37 0)
+      (effects (font (size 1.27 1.27)) hide)
+    )
+    (pin "1")
+    (pin "2")
+    (pin "3")
+    (pin "4")
+  )
+  (symbol (lib_id "power:GND") (at 161.29 66.04 0) (unit 1)
+    (in_bom yes) (on_board yes) (fields_autoplaced)
+    (property "Reference" "#PWR?" (id 0) (at 161.29 72.39 0)
+      (effects (font (size 1.27 1.27)) hide)
+    )
+    (property "Value" "GND" (id 1) (at 161.29 71.12 0))
+    (property "Footprint" "" (id 2) (at 161.29 66.04 0)
+      (effects (font (size 1.27 1.27)) hide)
+    )
+    (property "Datasheet" "" (id 3) (at 161.29 66.04 0)
+      (effects (font (size 1.27 1.27)) hide)
+    )
+    (pin "1")
+  )
+  (symbol (lib_id "Connector:Conn_01x04_Male") (at 153.67 58.42 0) (unit 1)
+    (in_bom yes) (on_board yes) (fields_autoplaced)
+    (property "Reference" "J?" (id 0) (at 154.305 50.8 0))
+    (property "Value" "Conn_01x04_Male" (id 1) (at 154.305 53.34 0))
+    (property "Footprint" "Connector_PinHeader_2.54mm:PinHeader_1x04_P2.54mm_Horizontal" (id 2) (at 153.67 58.42 0)
+      (effects (font (size 1.27 1.27)) hide)
+    )
+    (property "Datasheet" "~" (id 3) (at 153.67 58.42 0)
+      (effects (font (size 1.27 1.27)) hide)
+    )
+    (pin "1")
+    (pin "2")
+    (pin "3")
+    (pin "4")
+  )
+  (symbol (lib_id "Connector:Conn_01x02_Male") (at 31.75 99.06 0) (unit 1)
+    (in_bom yes) (on_board yes) (fields_autoplaced)
+    (property "Reference" "J?" (id 0) (at 32.385 93.98 0))
+    (property "Value" "Conn_01x02_Male" (id 1) (at 32.385 96.52 0))
+    (property "Footprint" "Connector_PinSocket_2.54mm:PinSocket_1x02_P2.54mm_Horizontal" (id 2) (at 31.75 99.06 0)
+      (effects (font (size 1.27 1.27)) hide)
+    )
+    (property "Datasheet" "~" (id 3) (at 31.75 99.06 0)
+      (effects (font (size 1.27 1.27)) hide)
+    )
+    (pin "1")
+    (pin "2")
+  )
+  (symbol (lib_id "Connector:Conn_01x02_Male") (at 31.75 58.42 0) (unit 1)
+    (in_bom yes) (on_board yes) (fields_autoplaced)
+    (property "Reference" "J?" (id 0) (at 32.385 53.34 0))
+    (property "Value" "Conn_01x02_Male" (id 1) (at 32.385 55.88 0))
+    (property "Footprint" "Connector_Phoenix_MC_HighVoltage:PhoenixContact_MC_1,5_2-G-5.08_1x02_P5.08mm_Horizontal" (id 2) (at 31.75 58.42 0)
+      (effects (font (size 1.27 1.27)) hide)
+    )
+    (property "Datasheet" "~" (id 3) (at 31.75 58.42 0)
+      (effects (font (size 1.27 1.27)) hide)
+    )
+    (pin "1")
+    (pin "2")
+  )
+  (symbol (lib_id "Connector:Conn_01x02_Male") (at 99.06 39.37 0) (unit 1)
+    (in_bom yes) (on_board yes) (fields_autoplaced)
+    (property "Reference" "J?" (id 0) (at 99.695 34.29 0))
+    (property "Value" "Conn_01x02_Male" (id 1) (at 99.695 36.83 0))
+    (property "Footprint" "Connector_PinSocket_2.54mm:PinSocket_1x02_P2.54mm_Horizontal" (id 2) (at 99.06 39.37 0)
+      (effects (font (size 1.27 1.27)) hide)
+    )
+    (property "Datasheet" "~" (id 3) (at 99.06 39.37 0)
+      (effects (font (size 1.27 1.27)) hide)
+    )
+    (pin "1")
+    (pin "2")
+  )
+  (symbol (lib_id "Connector:Conn_01x02_Male") (at 99.06 58.42 0) (unit 1)
+    (in_bom yes) (on_board yes)
+    (property "Reference" "J?" (id 0) (at 99.695 53.34 0))
+    (property "Value" "Conn_01x02_Male" (id 1) (at 99.695 55.88 0))
+    (property "Footprint" "Connector_PinSocket_2.54mm:PinSocket_1x02_P2.54mm_Horizontal" (id 2) (at 99.06 58.42 0)
+      (effects (font (size 1.27 1.27)) hide)
+    )
+    (property "Datasheet" "~" (id 3) (at 99.06 58.42 0)
+      (effects (font (size 1.27 1.27)) hide)
+    )
+    (pin "1")
+    (pin "2")
+  )
+  (symbol (lib_id "power:GND") (at 161.29 46.99 0) (unit 1)
+    (in_bom yes) (on_board yes) (fields_autoplaced)
+    (property "Reference" "#PWR?" (id 0) (at 161.29 53.34 0)
+      (effects (font (size 1.27 1.27)) hide)
+    )
+    (property "Value" "GND" (id 1) (at 161.29 52.07 0))
+    (property "Footprint" "" (id 2) (at 161.29 46.99 0)
+      (effects (font (size 1.27 1.27)) hide)
+    )
+    (property "Datasheet" "" (id 3) (at 161.29 46.99 0)
+      (effects (font (size 1.27 1.27)) hide)
+    )
+    (pin "1")
+  )
+  (symbol (lib_id "Connector:Conn_01x02_Male") (at 31.75 39.37 0) (unit 1)
+    (in_bom yes) (on_board yes)
+    (property "Reference" "J?" (id 0) (at 32.385 34.29 0))
+    (property "Value" "Conn_01x02_Male" (id 1) (at 32.385 36.83 0))
+    (property "Footprint" "Connector_Phoenix_MC_HighVoltage:PhoenixContact_MC_1,5_2-G-5.08_1x02_P5.08mm_Horizontal" (id 2) (at 31.75 39.37 0)
+      (effects (font (size 1.27 1.27)) hide)
+    )
+    (property "Datasheet" "~" (id 3) (at 31.75 39.37 0)
+      (effects (font (size 1.27 1.27)) hide)
+    )
+    (pin "1")
+    (pin "2")
+  )
 )

Commit message: 1st drawing
Parts:
- added H1, H2, H3, H4: MountingHole_Pad, MountingHole:MountingHole_2.2mm_M2_ISO14580_Pad, symbol Mechanical:MountingHole_Pad
- added J10, J11: Conn_01x02_Male, Connector_PinSocket_2.54mm:PinSocket_1x02_P2.54mm_Horizontal, symbol Connector:Conn_01x02_Male
- added R1: 120, Resistor_SMD:R_0805_2012Metric, symbol Device:R
- added SW1: NDS-01-V, DIP762W60P254L390H705Q2N, symbol NDS-01-V:NDS-01-V
- gave numbers to parts that had none: 9
Connections:
- net GND: now also H1.1, H2.1, H3.1, H4.1, J10.2 (Pin_2), J11.2 (Pin_2)
- net CANL: now reaches J4.1 (Pin_1)
- net CANL: now also J3.1 (Pin_1), J5.1 (Pin_1), SW1.1
- net CANH: now reaches J4.2 (Pin_2)
- net CANH: now also J3.2 (Pin_2), J5.2 (Pin_2), R1.2
- net +5V: now reaches J8.1 (Pin_1)
- net +5V: now also J9.1 (Pin_1), J10.1 (Pin_1)
- net COD_GAUCHE_A: now reaches J8.2 (Pin_2)
- net COD_GAUCHE_B: now reaches J8.3 (Pin_3)
- net COD_DROIT_A: now reaches J9.2 (Pin_2)
- net COD_DROIT_B: now reaches J9.3 (Pin_3)
- net Vbat_puissance: now reaches J2.1 (Pin_1)
- net Moteur_Gauche_P: now reaches J6.1 (Pin_1)
- net Moteur_Gauche_N: now reaches J6.2 (Pin_2)
- net Moteur_Droit_P: now reaches J7.1 (Pin_1)
- net Moteur_Droit_N: now reaches J7.2 (Pin_2)
- net Vbat_logic: now reaches J1.1 (Pin_1)
- new net: R1.1, SW1.2
- new net +3.3V: J11.1 (Pin_1)
Other:
- note added: "Mécanique"
- note added: "TEST TENSION"
