File: Conception/IHM.kicad_sch (KiCad schematic)
At the start: 0 parts

Commit message: MAJ
Other:
- company: AstroMonkeys -> (none)
Changed lines of the file:
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@@
 (kicad_sch (version 20211123) (generator eeschema)
   (paper "A4")
-  (title_block
-    (rev "0.1")
-    (company "AstroMonkeys")
-  )
 )

Commit message: 1st drawing
Parts:
- added D1, D12, D2, D3, D4, D5, D7, D9: SML-210PTT86, LED_SMD:LED_0805_2012Metric, symbol Device:LED
- added D10, D6, D8: SML-210LTT86, LED_SMD:LED_0805_2012Metric, symbol Device:LED
- added D11, D13, D14: LED, LED_SMD:LED_0805_2012Metric, symbol Device:LED
- added R10, R11, R12, R13, R14, R15, R16, R17, R8, R9: R, Resistor_SMD:R_0805_2012Metric, symbol Device:R
- added R18, R19, R2, R3, R4, R5: 10k, Resistor_SMD:R_0805_2012Metric, symbol Device:R
- added R6, R7: 1.2k, Resistor_SMD:R_0805_2012Metric, symbol Device:R
- added SW2, SW3, SW4, SW5, SW6, SW7: NDS-01-V, DIP762W60P254L390H705Q2N, symbol NDS-01-V:NDS-01-V
Connections:
- new net: D9.1 (K), R12.2
- new net: D4.1 (K), R9.2
- new net: D13.1 (K), R16.2
- new net: D10.1 (K), R13.2
- new net: D14.1 (K), R17.2
- new net: D12.1 (K), R15.2
- new net: D3.1 (K), R8.2
- new net: D7.2 (A), D8.1 (K)
- new net: D7.1 (K), D8.2 (A), R11.2
- new net: D11.1 (K), R14.2
- new net: D2.1 (K), R7.2
- new net: D5.1 (K), D6.2 (A), R10.2
- new net: D1.1 (K), R6.2
- new net: D5.2 (A), D6.1 (K)
- new net +3.3V: D4.2 (A), R18.1, R19.1, R2.1, R3.1, R4.1, R5.1, SW2.1, SW3.1, SW4.1, SW5.1, SW6.1, SW7.1
- new net +5V: D3.2 (A)
- new net Debug_0: SW2.2
- new net Debug_1: SW4.2
- new net Debug_2: SW6.2
- new net Debug_3: SW7.2
- new net Debug_4: SW3.2
- new net Debug_5: SW5.2
- new net GND: R10.1, R11.1, R12.1, R13.1, R14.1, R15.1, R16.1, R17.1, R18.2, R19.2, R2.2, R3.2, R4.2, R5.2, R6.1, R7.1, R8.1, R9.1
- new net LED_DEBUG_0: D9.2 (A)
- new net LED_DEBUG_1: D10.2 (A)
- new net LED_DEBUG_2: D11.2 (A)
- new net LED_DEBUG_3: D12.2 (A)
- new net LED_DEBUG_4: D13.2 (A)
- new net LED_DEBUG_5: D14.2 (A)
- new net Vbat_logic: D1.2 (A)
- new net Vbat_puissance: D2.2 (A)
Other:
- note added: "DEBUG LED"
- note added: "DEBUG SWITCH"
- note added: "INFO LED"
- note added: "LED ALIM"
- note added: "LED MOTEUR"
- note added: "SML-210PTT86 => LED VERTE SML-210LTT86 => LED ROUGE"
